Commit message: alice_v2

File: src/alice_description/urdf/alice_v2.xacro (robot description, xacro)
@@ -4,7 +4,8 @@
     <gazebo>
         <plugin name="gazebo_ros_control" filename="libgazebo_ros_control.so">
+            <robotNamespace>/alice</robotNamespace>
         </plugin>
     </gazebo>
-    <!-- <gazebo reference="base_cyllinder">
+    <gazebo reference="base_cyllinder">
         <turnGravityOff>true</turnGravityOff>
     </gazebo>
@@ -23,5 +24,5 @@
     <gazebo reference="camera_link">
         <turnGravityOff>true</turnGravityOff>
-    </gazebo> -->
+    </gazebo>
     <!-- The rescaling of 0.001 is necessary because gazebo takes all inputs as meters -->
     <!-- Meaning 100mm will be seen as 100m, hence rescaling is needed -->
@@ -207,5 +208,5 @@
         <parent link="wrist_link" />
         <child link="camera_link" />
-        <origin rpy="0 0 0" xyz="0 0 0.073" />
+        <origin rpy="1.5707 1.5707 1.5707" xyz="0.038 0 0.03" />
     </joint>
     <gazebo reference="base_cyllinder">

Commit message: routine save

File: src/alice_description/urdf/alice_v2.xacro (robot description, xacro)
@@ -140,4 +140,25 @@
                 izz="1.4021e-05" />
         </inertial>
+    </link>
+    <link name="Camera_connect_link">
+        <visual>
+            <geometry>
+                <box size="0.0 0.0 0.0"/>
+            </geometry>
+            <material name="black" />
+            <origin rpy="0 0 0" xyz="0 0 0" />
+        </visual>
+        <inertial>
+            <origin rpy="0 0 0" xyz="0 0 0" />
+            <mass value="100" />
+            <inertia ixx="0.0702" ixy="0" ixz="0" iyy="0.0702" iyz="0"
+                izz="0.1404" />
+        </inertial>
+        <collision>
+            <geometry>
+                <cylinder length="0.001" radius="0.053" />
+            </geometry>
+            <origin rpy="0 0 0" xyz="0 0 0" />
+        </collision>
     </link>
     <!-- Create the link (or like item) -->

Commit message: new moveit

File: src/alice_description/urdf/alice_v2.xacro (robot description, xacro)
@@ -141,5 +141,5 @@
         </inertial>
     </link>
-    <!-- <link name="wrist_link_roll">
+    <link name="wrist_link_roll">
         <visual>
             <geometry>
@@ -160,5 +160,5 @@
             <inertia ixx="0.000348958333333" ixy="0" ixz="0" iyy="0.000348958333333" iyz="0" izz="3.125e-05" />
         </inertial>
-    </link> -->
+    </link>
     <!-- Add alternative way to look at your camera -->
     <!-- We need to turn it 90 degrees in yaw, CCW -->

File: src/alice_moveit/config/gazebo_alice.urdf (robot description, URDF)
Before this commit: robot alice, 8 links, 7 joints
Links:
- removed link base_cyllinder
- removed link camera_link_optical
- removed link wrist_link
- added link base_link, mass 100; collision cylinder length=0.001 radius=0.053; visual cylinder length=0.003 radius=.053
- added link camera_bottom_screw_frame
- added link camera_mount, mass 0.059; collision mesh filename=package://alice_description/stl/alice_camera_mount_v3.stl scale=0.001 0.001 0.001; visual mesh filename=package://alice_description/stl/alice_camera_mount_v3.stl scale=0.001 0.001 0.001
- added link wrist_link_pitch, mass 0.059; collision mesh filename=package://alice_description/stl/braccio_wrist_pitch.stl scale=0.001 0.001 0.001; visual mesh filename=package://alice_description/stl/braccio_wrist_pitch.stl scale=0.001 0.001 0.001
- added link wrist_link_roll, mass 0.059; collision mesh filename=package://alice_description/stl/braccio_wrist_roll.stl scale=0.001 0.001 0.001; visual mesh filename=package://alice_description/stl/braccio_wrist_roll.stl scale=0.001 0.001 0.001
- link camera_link: geometry collision box size=0.02505 0.09 0.025; visual mesh filename=package://realsense2_description/meshes/d435.dae
Joints:
- removed joint camera_optical_joint
- added joint camera_link_joint: type fixed, parent camera_bottom_screw_frame, child camera_link, origin xyz=0.010600000000000002 0.0175 0.0125 rpy=0 0 0
- added joint camera_mount_joint: type fixed, parent wrist_link_roll, child camera_mount, origin xyz=0.006 0.013 0.046 rpy=1.5708 -3.14 3.14
- added joint wrist_roll_joint: type revolute, parent wrist_link_pitch, child wrist_link_roll, origin xyz=-0.0007 -0.003 0.111 rpy=0 1.5708 0, axis 1 0 0, limit lower=0 upper=3.1416 effort=1.0 velocity=1.0
- joint base_joint: parent base_cyllinder -> base_link
- joint camera_joint: child camera_link -> camera_bottom_screw_frame; origin xyz=0 0 0.073 rpy=0 0 0 -> xyz=0.013 0.0507 0.043 rpy=0 4.71238 1.5708; parent wrist_link -> camera_mount
- joint world_joint: child base_cyllinder -> base_link
- joint wrist_pitch_joint: child wrist_link -> wrist_link_pitch
