Commit message: Update

File: src/alice_description/urdf/alice_v1.xacro (robot description, xacro)
@@ -4,8 +4,7 @@
     <gazebo>
         <plugin name="gazebo_ros_control" filename="libgazebo_ros_control.so">
-            <robotNamespace>/alice</robotNamespace>
         </plugin>
     </gazebo>
-    <gazebo reference="base_cyllinder">
+    <!-- <gazebo reference="base_cyllinder">
         <turnGravityOff>true</turnGravityOff>
     </gazebo>
@@ -24,5 +23,7 @@
     <gazebo reference="camera_link">
         <turnGravityOff>true</turnGravityOff>
-    </gazebo>
+    </gazebo> -->
+    <!-- The rescaling of 0.001 is necessary because gazebo takes all inputs as meters -->
+    <!-- Meaning 100mm will be seen as 100m, hence rescaling is needed -->
     <!-- The base link is the cyllinder at the bottom-->
     <link name="base_cyllinder">
@@ -36,7 +37,7 @@
         <inertial>
             <origin rpy="0 0 0" xyz="0 0 0" />
-            <mass value="2" />
-            <inertia ixx="0.015" ixy="0" ixz="0" iyy="0.00666666666667" iyz="0"
-                izz="0.0216666666667" />
+            <mass value="100" />
+            <inertia ixx="0.0702" ixy="0" ixz="0" iyy="0.0702" iyz="0"
+                izz="0.1404" />
         </inertial>
         <collision>
@@ -65,7 +66,7 @@
         <inertial>
             <origin rpy="0 0 3.1416" xyz="0 0.004 0" />
-            <mass value="1" />
-            <inertia ixx="0.015" ixy="0" ixz="0" iyy="0.00666666666667" iyz="0"
-                izz="0.0216666666667" />
+            <mass value="0.262" />
+            <inertia ixx="4.0242e-04" ixy="0" ixz="0" iyy="4.0242e-04" iyz="0"
+                izz="3.6797e-04" />
         </inertial>
     </link>
@@ -88,7 +89,7 @@
         <inertial>
             <origin rpy="0 0 0" xyz="-0.0045 0.0055 -0.026" />
-            <mass value="0.1" />
-            <inertia ixx="0.000348958333333" ixy="0" ixz="0" iyy="0.000348958333333" iyz="0"
-                izz="3.125e-05" />
+            <mass value="0.126" />
+            <inertia ixx="0.0003385" ixy="0" ixz="0" iyy="0.0003173" iyz="0"
+                izz="0.00004818" />
         </inertial>
     </link>
@@ -111,7 +112,7 @@
         <inertial>
             <origin rpy="0 0 0" xyz="-0.0045 0.005 -0.025" />
-            <mass value="0.1" />
-            <inertia ixx="0.000348958333333" ixy="0" ixz="0" iyy="0.000348958333333" iyz="0"
-                izz="3.125e-05" />
+            <mass value="0.119" />
+            <inertia ixx="0.0003385" ixy="0" ixz="0" iyy="0.0003173" iyz="0"
+                izz="0.00004818" />
         </inertial>
     </link>
@@ -134,7 +135,7 @@
         <inertial>
             <origin rpy="0 0 0" xyz="0.003 -0.0004 -0.024" />
-            <mass value="0.1" />
-            <inertia ixx="0.000348958333333" ixy="0" ixz="0" iyy="0.000348958333333" iyz="0"
-                izz="3.125e-05" />
+            <mass value="0.059" />
+            <inertia ixx="1.5897e-05" ixy="0" ixz="0" iyy="2.5056e-05" iyz="0"
+                izz="1.4021e-05" />
         </inertial>
     </link>
@@ -155,7 +156,7 @@
         </collision>
         <inertial>
-            <mass value="0.1" />
-            <inertia ixx="0.000348958333333" ixy="0" ixz="0" iyy="0.000348958333333" iyz="0"
-                izz="3.125e-05" />
+            <mass value="0.072" />
+            <inertia ixx="0.0" ixy="0" ixz="0" iyy="0" iyz="0"
+                izz="0" />
         </inertial>
     </link>

File: src/alice_moveit/config/gazebo_alice.urdf (robot description, URDF)
Before this commit: robot alice, 8 links, 7 joints
Links:
- removed link realsense_camera
- removed link realsense_camera_optical
- added link camera_link, mass 0.072; collision box size=0.08 0.02 0.02; visual box size=0.09 0.025 0.025
- added link camera_link_optical
- link base_cyllinder: mass 2 -> 100
- link elbow_link: mass 0.1 -> 0.119
- link rotating_base: mass 1 -> 0.262
- link shoulder_link: mass 0.1 -> 0.126
- link wrist_link: mass 0.1 -> 0.059
Joints:
- joint camera_joint: child realsense_camera -> camera_link; origin xyz=0 0 0.073 rpy=-1.5708 0 0 -> xyz=0 0 0.073 rpy=0 0 0
- joint camera_optical_joint: child realsense_camera_optical -> camera_link_optical; origin xyz=0 0 0 rpy=-1.57079632679 0 -1.57079632679 -> xyz=0 0 0 rpy=-3.14 -1.5707 -1.5707; parent realsense_camera -> camera_link

Commit message: update

File: src/alice_description/urdf/alice_v1.xacro (robot description, xacro)
@@ -6,5 +6,5 @@
         </plugin>
     </gazebo>
-    <!-- <gazebo reference="base_cyllinder">
+    <gazebo reference="base_cyllinder">
         <turnGravityOff>true</turnGravityOff>
     </gazebo>
@@ -18,10 +18,10 @@
         <turnGravityOff>true</turnGravityOff>
     </gazebo>
-    <gazebo reference="wrist_link">
-        <turnGravityOff>true</turnGravityOff>
-    </gazebo>
-    <gazebo reference="camera_link">
-        <turnGravityOff>true</turnGravityOff>
-    </gazebo> -->
+    <gazebo reference="wrist_link_pitch">
+        <turnGravityOff>true</turnGravityOff>
+    </gazebo>
+    <gazebo reference="wrist_link_roll">
+        <turnGravityOff>true</turnGravityOff>
+    </gazebo>
     <!-- The rescaling of 0.001 is necessary because gazebo takes all inputs as meters -->
     <!-- Meaning 100mm will be seen as 100m, hence rescaling is needed -->
@@ -32,5 +32,5 @@
                 <cylinder length="0.003" radius=".053" />
             </geometry>
-            <material name="black" />
+            <material name="orange" />
             <origin rpy="0 0 0" xyz="0 0 0" />
         </visual>
@@ -117,5 +117,5 @@
         </inertial>
     </link>
-    <link name="wrist_link">
+    <link name="wrist_link_pitch">
         <visual>
             <geometry>
@@ -140,6 +140,26 @@
         </inertial>
     </link>
+    <link name="wrist_link_roll">
+        <visual>
+            <geometry>
+                <mesh filename="package://alice_description/stl/braccio_wrist_roll.stl" scale="0.001 0.001 0.001" />
+            </geometry>
+            <material name="white" />
+            <origin rpy="0 0 0" xyz="0 0 0" />
+        </visual>
+        <collision>
+            <geometry>
+                <mesh filename="package://alice_description/stl/braccio_wrist_roll.stl" scale="0.001 0.001 0.001" />
+            </geometry>
+            <origin rpy="0 0 0" xyz="0 0 0" />
+        </collision>
+        <inertial>
+            <origin rpy="0 0 0" xyz="0 0 0" />
+            <mass value="0.059" />
+            <inertia ixx="0.000348958333333" ixy="0" ixz="0" iyy="0.000348958333333" iyz="0" izz="3.125e-05" />
+        </inertial>
+    </link>
     <!-- Create the link (or like item) -->
-    <link name="camera_link">
+    <!-- <link name="camera_link">
         <visual>
             <origin xyz="0 0 0" rpy="0 0 0" />
@@ -160,8 +180,8 @@
                 izz="0" />
         </inertial>
-    </link>
+    </link> -->
     <!-- Add alternative way to look at your camera -->
     <!-- We need to turn it 90 degrees in yaw, CCW -->
-    <link name="camera_link_optical">
+    <!-- <link name="camera_link_optical">
     </link>
     <joint name="camera_optical_joint" type="fixed">
@@ -169,5 +189,5 @@
         <child link="camera_link_optical" />
         <origin xyz="0 0 0" rpy="-3.14 -1.5707 -1.5707" />
-    </joint>
+    </joint> -->
     <!-- Add alternative way to look at your camera -->
     <!-- Base joint is the rotating thing -->
@@ -201,12 +221,20 @@
         <origin rpy="-1.5708 0 0" xyz="0 0 0.125" />
         <parent link="elbow_link" />
-        <child link="wrist_link" />
-        <dynamics damping="0.1" friction="0.001" />
-    </joint>
-    <joint name="camera_joint" type="fixed">
-        <parent link="wrist_link" />
+        <child link="wrist_link_pitch" />
+        <dynamics damping="0.1" friction="0.001" />
+    </joint>
+    <joint name="wrist_roll_joint" type="revolute">
+        <axis xyz="0 1 0" />
+        <limit effort="1.0" lower="0" upper="3.1416" velocity="1.0" />
+        <origin rpy="0 0 0" xyz="0.006 0 0.062" />
+        <parent link="wrist_link_pitch" />
+        <child link="wrist_link_roll" />
+        <dynamics damping="0.1" friction="0.001" />
+    </joint>
+    <!-- <joint name="camera_joint" type="fixed">
+        <parent link="wrist_link_roll" />
         <child link="camera_link" />
         <origin rpy="0 0 0" xyz="0 0 0.073" />
-    </joint>
+    </joint> -->
     <gazebo reference="base_cyllinder">
         <mu1>1</mu1>
@@ -219,5 +247,5 @@
         <mu2>1</mu2>
         <selfCollide>true</selfCollide>
-        <material>Gazebo/Green</material>
+        <material>Gazebo/Orange</material>
     </gazebo>
     <gazebo reference="shoulder_link">
@@ -231,16 +259,22 @@
         <mu2>1</mu2>
         <selfCollide>true</selfCollide>
-        <material>Gazebo/Blue</material>
-    </gazebo>
-    <gazebo reference="wrist_link">
-        <mu1>1</mu1>
-        <mu2>1</mu2>
-        <selfCollide>true</selfCollide>
-        <material>Gazebo/Red</material>
-    </gazebo>
-    <gazebo reference="camera_link">
+        <material>Gazebo/Orange</material>
+    </gazebo>
+    <gazebo reference="wrist_link_pitch">
+        <mu1>1</mu1>
+        <mu2>1</mu2>
+        <selfCollide>true</selfCollide>
+        <material>Gazebo/Orange</material>
+    </gazebo>
+    <gazebo reference="wrist_link_roll">
+        <mu1>1</mu1>
+        <mu2>1</mu2>
+        <selfCollide>true</selfCollide>
+        <material>Gazebo/White</material>
+    </gazebo>
+    <!-- <gazebo reference="camera_link">
         <selfCollide>true</selfCollide>
         <material>Gazebo/Black</material>
-    </gazebo>
+    </gazebo> -->
     <!-- Specify colors-->
     <material name="orange">

File: src/alice_description/urdf/alice_v2.xacro (robot description, xacro)
@@ -141,46 +141,24 @@
         </inertial>
     </link>
-    <link name="Camera_connect_link">
-        <visual>
-            <geometry>
-                <box size="0.0 0.0 0.0"/>
-            </geometry>
-            <material name="black" />
-            <origin rpy="0 0 0" xyz="0 0 0" />
-        </visual>
-        <inertial>
-            <origin rpy="0 0 0" xyz="0 0 0" />
-            <mass value="100" />
-            <inertia ixx="0.0702" ixy="0" ixz="0" iyy="0.0702" iyz="0"
-                izz="0.1404" />
-        </inertial>
-        <collision>
-            <geometry>
-                <cylinder length="0.001" radius="0.053" />
-            </geometry>
-            <origin rpy="0 0 0" xyz="0 0 0" />
-        </collision>
-    </link>
-    <!-- Create the link (or like item) -->
-    <link name="camera_link">
-        <visual>
-            <origin xyz="0 0 0" rpy="0 0 0" />
-            <geometry>
-                <box size="0.09 0.025 0.025" />
-            </geometry>
-            <material name="black" />
-        </visual>
-        <collision>
-            <origin xyz="0 0 0" rpy="0 0 0" />
-            <geometry>
-                <box size="0.08 0.02 0.02" />
-            </geometry>
-        </collision>
-        <inertial>
-            <mass value="0.072" />
-            <inertia ixx="0.0" ixy="0" ixz="0" iyy="0" iyz="0"
-                izz="0" />
-        </inertial>
-    </link>
+    <!-- <link name="wrist_link_roll">
+        <visual>
+            <geometry>
+                <mesh filename="package://alice_description/stl/braccio_wrist_roll.stl" scale="0.001 0.001 0.001" />
+            </geometry>
+            <material name="white" />
+            <origin rpy="0 0 0" xyz="0.006 0 0.0" />
+        </visual>
+        <collision>
+            <geometry>
+                <mesh filename="package://alice_description/stl/braccio_wrist_roll.stl" scale="0.001 0.001 0.001" />
+            </geometry>
+            <origin rpy="0 0 0" xyz="0.006 0 0.0" />
+        </collision>
+        <inertial>
+            <origin rpy="0 0 0" xyz="0.006 0 0.0" />
+            <mass value="0.1" />
+            <inertia ixx="0.000348958333333" ixy="0" ixz="0" iyy="0.000348958333333" iyz="0" izz="3.125e-05" />
+        </inertial>
+    </link> -->
     <!-- Add alternative way to look at your camera -->
     <!-- We need to turn it 90 degrees in yaw, CCW -->
@@ -226,9 +204,12 @@
         <dynamics damping="0.1" friction="0.001" />
     </joint>
-    <joint name="camera_joint" type="fixed">
+    <!-- <joint name="wrist_roll_joint" type="revolute">
+        <axis xyz="0 0 -1" />
+        <limit effort="1.0" lower="0.0" upper="3.1416" velocity="1.0" />
+        <origin rpy="0 0 1.5708" xyz="0 0.0 0.06" />
         <parent link="wrist_link" />
-        <child link="camera_link" />
-        <origin rpy="1.5707 1.5707 1.5707" xyz="0.038 0 0.03" />
-    </joint>
+        <child link="wrist_link_roll" />
+        <dynamics damping="0.1" friction="0.001" />
+    </joint> -->
     <gazebo reference="base_cyllinder">
         <mu1>1</mu1>
@@ -264,4 +245,8 @@
         <selfCollide>true</selfCollide>
         <material>Gazebo/Black</material>
+    </gazebo>
+    <gazebo reference="wrist_link_roll">
+        <selfCollide>true</selfCollide>
+        <material>Gazebo/White</material>
     </gazebo>
     <!-- Specify colors-->

Commit message: Finished URDF

File: src/alice_description/urdf/alice_v1.xacro (robot description, xacro)
@@ -149,5 +149,5 @@
             </geometry>
             <material name="white" />
-            <origin rpy="0 0 0" xyz="0 0 0" />
+            <origin rpy="0 0 0" xyz="0 -0.0205 -0.039" />
         </visual>
         <collision>
@@ -248,7 +248,8 @@
     </joint>
     <joint name="wrist_roll_joint" type="revolute">
-        <axis xyz="0 0 1" />
+        <axis xyz="1 0 0" />
         <limit effort="1.0" lower="0" upper="3.1416" velocity="1.0" />
-        <origin rpy="0 0 1.5708" xyz="-0.001 0.003 0.062" />
+        <!-- <origin rpy="0 1.5708 0" xyz="-0.019 0.012 0.1117" /> -->
+        <origin rpy="0 1.5708 0" xyz="-0.0007 -0.003 0.111"/>
         <parent link="wrist_link_pitch" />
         <child link="wrist_link_roll" />
@@ -256,5 +257,5 @@
     </joint>
     <joint name="camera_mount_joint" type="fixed">
-        <origin rpy="0 1.5708 1.5708" xyz="0.035 -0.001 0.042" />
+        <origin rpy="1.5708 -3.14 3.14" xyz="0.006 0.013 0.046" />
         <parent link="wrist_link_roll" />
         <child link="camera_mount" />
@@ -265,4 +266,10 @@
         <origin rpy="0 0 0" xyz="0 0 0.073" />
     </joint> -->
+    <!-- Add the D435 Camera -->
+    <xacro:arg name="use_nominal_extrinsics" default="false" />
+    <xacro:include filename="$(find realsense2_description)/urdf/_d435.urdf.xacro"/>
+    <xacro:sensor_d435 parent="camera_mount" use_nominal_extrinsics="$(arg use_nominal_extrinsics)">
+        <origin xyz="0.013 0.0507 0.043" rpy="0 4.71238 1.5708" scale = " 0.001 0.001 0.001" />
+    </xacro:sensor_d435>
     <gazebo reference="base_cyllinder">
         <mu1>1</mu1>
@@ -301,7 +308,7 @@
         <material>Gazebo/White</material>
     </gazebo>
-    <gazebo reference="camera_mount_link">
-        <selfCollide>true</selfCollide>
-        <material>Gazebo/Green</material>
+    <gazebo reference="camera_mount">
+        <selfCollide>true</selfCollide>
+        <material>Gazebo/Black</material>
     </gazebo>
     <!-- <gazebo reference="camera_link">

Commit message: Fixed moveit

File: src/alice_description/urdf/alice_v1.xacro (robot description, xacro)
@@ -4,4 +4,5 @@
     <gazebo>
         <plugin name="gazebo_ros_control" filename="libgazebo_ros_control.so">
+            <robotNamespace>/alice</robotNamespace>
         </plugin>
     </gazebo>
@@ -168,5 +169,5 @@
                 <mesh filename="package://alice_description/stl/alice_camera_mount_v3.stl" scale="0.001 0.001 0.001" />
             </geometry>
-            <material name="green" />
+            <material name="black" />
             <origin rpy="0 0 0" xyz="0 0 0" />
         </visual>
@@ -250,5 +251,4 @@
         <axis xyz="1 0 0" />
         <limit effort="1.0" lower="0" upper="3.1416" velocity="1.0" />
-        <!-- <origin rpy="0 1.5708 0" xyz="-0.019 0.012 0.1117" /> -->
         <origin rpy="0 1.5708 0" xyz="-0.0007 -0.003 0.111"/>
         <parent link="wrist_link_pitch" />
@@ -261,9 +261,4 @@
         <child link="camera_mount" />
     </joint>
-    <!-- <joint name="camera_joint" type="fixed">
-        <parent link="wrist_link_roll" />
-        <child link="camera_link" />
-        <origin rpy="0 0 0" xyz="0 0 0.073" />
-    </joint> -->
     <!-- Add the D435 Camera -->
     <xacro:arg name="use_nominal_extrinsics" default="false" />
@@ -420,3 +415,13 @@
         </actuator>
     </transmission>
+    <transmission name="trans_wrist_roll_joint">
+        <type>transmission_interface/SimpleTransmission</type>
+        <joint name="wrist_roll_joint">
+            <hardwareInterface>hardware_interface/EffortJointInterface</hardwareInterface>
+        </joint>
+        <actuator name="wrist_roll_joint_motor">
+            <hardwareInterface>hardware_interface/EffortJointInterface</hardwareInterface>
+            <mechanicalReduction>1</mechanicalReduction>
+        </actuator>
+    </transmission>
 </robot>

Commit message: fixed real-life controls

File: src/alice_description/urdf/alice_v1.xacro (robot description, xacro)
@@ -251,5 +251,5 @@
         <axis xyz="1 0 0" />
         <limit effort="1.0" lower="0" upper="3.1416" velocity="1.0" />
-        <origin rpy="0 1.5708 0" xyz="-0.0007 -0.003 0.111"/>
+        <origin rpy="3.14159 1.5708 0" xyz="-0.0007 -0.003 0.111"/>
         <parent link="wrist_link_pitch" />
         <child link="wrist_link_roll" />
@@ -326,5 +326,5 @@
         <parent link="world" />
         <child link="base_link" />
-        <origin rpy="0.0 0.0 0.0" xyz="0.0 0.0 0.0" />
+        <origin rpy="0 0.0 0.925025" xyz="0.0 0.0 0.0" />
     </joint>
     <!-- Gazebo reference for depth camera -->

File: src/alice_moveit/config/gazebo_alice.urdf (robot description, URDF)
Before this commit: robot alice, 10 links, 9 joints
Joints:
- joint world_joint: origin xyz=0.0 0.0 0.0 rpy=0.0 0.0 0.0 -> xyz=0.0 0.0 0.0 rpy=0.925025 0.0 0.0
- joint wrist_roll_joint: origin xyz=-0.0007 -0.003 0.111 rpy=0 1.5708 0 -> xyz=-0.0007 -0.003 0.111 rpy=3.14159 1.5708 0

Commit message: lagg

File: src/alice_description/urdf/alice_v1.xacro (robot description, xacro)
@@ -251,5 +251,5 @@
         <axis xyz="1 0 0" />
         <limit effort="1.0" lower="0" upper="3.1416" velocity="1.0" />
-        <origin rpy="3.14159 1.5708 0" xyz="-0.0007 -0.003 0.111"/>
+        <origin rpy="0 1.5708 0" xyz="-0.0007 -0.003 0.111"/>
         <parent link="wrist_link_pitch" />
         <child link="wrist_link_roll" />
@@ -326,5 +326,5 @@
         <parent link="world" />
         <child link="base_link" />
-        <origin rpy="0 0.0 0.925025" xyz="0.0 0.0 0.0" />
+        <origin rpy="0 0 -0.575959" xyz="0.0 0.0 0.0" />
     </joint>
     <!-- Gazebo reference for depth camera -->

File: src/alice_moveit/config/gazebo_alice.urdf (robot description, URDF)
Before this commit: robot alice, 10 links, 9 joints
Joints:
- joint world_joint: origin xyz=0.0 0.0 0.0 rpy=0.925025 0.0 0.0 -> xyz=0.0 0.0 0.0 rpy=0 0.0 0.925025

Commit message: Synced with real-life robot

File: src/alice_description/urdf/alice_v1.xacro (robot description, xacro)
@@ -226,5 +226,5 @@
     <joint name="shoulder_joint" type="revolute">
         <axis xyz="1 0 0" />
-        <limit effort="1.0" lower="0.2618" upper="2.8798" velocity="1.0" />
+        <limit effort="1.0" lower="0.523599" upper="2.61799" velocity="1.0" />
         <origin rpy="-1.5708 0 0" xyz="0 -.002 0.072" />
         <parent link="rotating_base" />
@@ -326,5 +326,5 @@
         <parent link="world" />
         <child link="base_link" />
-        <origin rpy="0 0 -0.575959" xyz="0.0 0.0 0.0" />
+        <origin rpy="0 0 2.56563" xyz="0.0 0.0 0.0" />
     </joint>
     <!-- Gazebo reference for depth camera -->

Commit message: only need check TF, otherwise good

File: src/alice_description/urdf/alice_v1.xacro (robot description, xacro)
@@ -326,5 +326,5 @@
         <parent link="world" />
         <child link="base_link" />
-        <origin rpy="0 0 2.56563" xyz="0.0 0.0 0.0" />
+        <origin rpy="0 0 2.35619" xyz="0.0 0.0 0.0" />
     </joint>
     <!-- Gazebo reference for depth camera -->
